Commit message: v1 PD control, updated urdf

File: diff_drive_real.urdf (robot description, URDF)
Before this commit: robot diff_drive, 5 links, 3 joints
Links:
- added link head, mass .156; collision box size=0.08255 0.1016 0.01; visual box size=0.08255 0.1016 0.01
- link base_link: geometry visual box size=0.025 0.03 0.04
- link extension: geometry visual box size=0.025 0.03 0.085
Joints:
- added joint extension_to_head: type fixed, parent extension, child head, origin xyz=0 0 0.043 rpy=0 0 0
